File: mm_power.kicad_sch (KiCad schematic)
At the start: 1 part, among them J5 Conn_01x02

Commit message: tp2
Parts:
- added C13, C14: 0.1uF, symbol Device:C
- added D1: LED, symbol Device:LED
- added R17: R, symbol Device:R
- added U4: LP5907MFX-3.3, Package_TO_SOT_SMD:SOT-23-5, symbol Regulator_Linear:LP5907MFX-3.3
Connections:
- net +BATT: now also C14.1, U4.1 (IN), U4.3 (EN)
- net GND: now also C13.2, C14.2, R17.2, U4.2 (GND)
- new net: D1.1 (K), R17.1
- new net +1V5: D1.2 (A)
- new net +3.3V: C13.1, U4.5 (OUT)
